File: hub.sch (EAGLE design)
At the start: 27 parts, among them U1 10118194-MICRO-USB, U2 LM3671MF-3.3/NOPBMF05A-M, U3 SN74LVC1T45DBVRDBV6-M, U4 SN74LVC1T45DBVRDBV6-M

Commit message: Polishing
Parts:
- R6: value 68 -> 220
Connections:
- net IO16 renamed GPIO16
- removed net IO17: JP7.6, U$2.IO17
- removed net IO19: JP7.2, U$2.IO19
- removed net IO25: JP7.5, U$2.IO25
- removed net IO26: JP7.7, U$2.IO26
- removed net IO27: JP7.9, U$2.IO27
- removed net IO33: JP7.3, U$2.IO33
- removed net IO4: JP7.8, U$2.IO4
- new net GPIO17: JP7.2, U$2.IO17
- new net GPIO25: JP7.7, U$2.IO25
- new net GPIO26: JP7.9, U$2.IO26
- new net GPIO27: JP7.8, U$2.IO27
- new net GPIO32: JP7.3, U$2.IO32
- new net GPIO33: JP7.5, U$2.IO33
- new net GPIO4: JP7.6, U$2.IO4
Changed lines of the file:
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@@
 <part name="JP5" library="jumper" library_urn="urn:adsk.eagle:library:252" deviceset="JP2E" device="" package3d_urn="urn:adsk.eagle:package:15452/1" value="LED Type"/>
 <part name="JP6" library="jumper" library_urn="urn:adsk.eagle:library:252" deviceset="JP2E" device="" package3d_urn="urn:adsk.eagle:package:15452/1" value="JTAG Enable"/>
-<part name="R6" library="rcl" library_urn="urn:adsk.eagle:library:334" deviceset="R-US_" device="R0805" package3d_urn="urn:adsk.eagle:package:23553/2" value="68"/>
+<part name="R6" library="rcl" library_urn="urn:adsk.eagle:library:334" deviceset="R-US_" device="R0805" package3d_urn="urn:adsk.eagle:package:23553/2" value="220"/>
 <part name="LED1" library="led" library_urn="urn:adsk.eagle:library:259" deviceset="LED" device="CHIPLED_0805" package3d_urn="urn:adsk.eagle:package:15821/2" value="Power"/>
 <part name="GND18" library="supply1" library_urn="urn:adsk.eagle:library:371" deviceset="GND" device=""/>
@@
 <instance part="JP6" gate="1" x="-48.26" y="17.78" smashed="yes">
 <attribute name="NAME" x="-52.07" y="17.78" size="1.778" layer="95" rot="R90"/>
-<attribute name="VALUE" x="-38.1" y="23.495" size="1.778" layer="96" rot="R180"/>
+<attribute name="VALUE" x="-45.72" y="26.035" size="1.778" layer="96" rot="R180"/>
 </instance>
 <instance part="U$2" gate="G$1" x="-7.62" y="5.08" smashed="yes"/>
@@
 </segment>
 </net>
-<net name="IO17" class="0">
+<net name="GPIO16" class="0">
+<segment>
+<pinref part="U$2" gate="G$1" pin="IO16"/>
+<wire x1="25.4" y1="-10.16" x2="35.56" y2="-10.16" width="0.1524" layer="91"/>
+<label x="38.1" y="-10.16" size="1.778" layer="95"/>
+</segment>
+</net>
+<net name="GPIO33" class="0">
+<segment>
+<pinref part="U$2" gate="G$1" pin="IO33"/>
+<wire x1="-27.94" y1="-2.54" x2="-35.56" y2="-2.54" width="0.1524" layer="91"/>
+<label x="-38.1" y="-2.54" size="1.778" layer="95" align="bottom-right"/>
+</segment>
+</net>
+<net name="GPIO27" class="0">
+<segment>
+<pinref part="U$2" gate="G$1" pin="IO27"/>
+<wire x1="-27.94" y1="-10.16" x2="-35.56" y2="-10.16" width="0.1524" layer="91"/>
+<label x="-38.1" y="-10.16" size="1.778" layer="95" align="bottom-right"/>
+</segment>
+</net>
+<net name="GPIO4" class="0">
+<segment>
+<pinref part="U$2" gate="G$1" pin="IO4"/>
+<wire x1="25.4" y1="-12.7" x2="35.56" y2="-12.7" width="0.1524" layer="91"/>
+<label x="38.1" y="-12.7" size="1.778" layer="95"/>
+</segment>
+</net>
+<net name="GPIO32" class="0">
+<segment>
+<pinref part="U$2" gate="G$1" pin="IO32"/>
+<wire x1="-27.94" y1="0" x2="-35.56" y2="0" width="0.1524" layer="91"/>
+<label x="-38.1" y="0" size="1.778" layer="95" align="bottom-right"/>
+</segment>
+</net>
+<net name="GPIO25" class="0">
+<segment>
+<pinref part="U$2" gate="G$1" pin="IO25"/>
+<wire x1="-27.94" y1="-5.08" x2="-35.56" y2="-5.08" width="0.1524" layer="91"/>
+<label x="-38.1" y="-5.08" size="1.778" layer="95" align="bottom-right"/>
+</segment>
+</net>
+<net name="GPIO26" class="0">
+<segment>
+<pinref part="U$2" gate="G$1" pin="IO26"/>
+<wire x1="-27.94" y1="-7.62" x2="-35.56" y2="-7.62" width="0.1524" layer="91"/>
+<label x="-38.1" y="-7.62" size="1.778" layer="95" align="bottom-right"/>
+</segment>
+</net>
+<net name="GPIO17" class="0">
 <segment>
 <pinref part="U$2" gate="G$1" pin="IO17"/>
 <wire x1="25.4" y1="-7.62" x2="35.56" y2="-7.62" width="0.1524" layer="91"/>
 <label x="38.1" y="-7.62" size="1.778" layer="95"/>
-</segment>
-</net>
-<net name="IO16" class="0">
-<segment>
-<pinref part="U$2" gate="G$1" pin="IO16"/>
-<wire x1="25.4" y1="-10.16" x2="35.56" y2="-10.16" width="0.1524" layer="91"/>
-<label x="38.1" y="-10.16" size="1.778" layer="95"/>
-</segment>
-</net>
-<net name="IO25" class="0">
-<segment>
-<pinref part="U$2" gate="G$1" pin="IO25"/>
-<wire x1="-27.94" y1="-5.08" x2="-35.56" y2="-5.08" width="0.1524" layer="91"/>
-<label x="-38.1" y="-5.08" size="1.778" layer="95" align="bottom-right"/>
-</segment>
-</net>
-<net name="IO26" class="0">
-<segment>
-<pinref part="U$2" gate="G$1" pin="IO26"/>
-<wire x1="-27.94" y1="-7.62" x2="-35.56" y2="-7.62" width="0.1524" layer="91"/>
-<label x="-38.1" y="-7.62" size="1.778" layer="95" align="bottom-right"/>
-</segment>
-</net>
-<net name="IO33" class="0">
-<segment>
-<pinref part="U$2" gate="G$1" pin="IO33"/>
-<wire x1="-27.94" y1="-2.54" x2="-35.56" y2="-2.54" width="0.1524" layer="91"/>
-<label x="-38.1" y="-2.54" size="1.778" layer="95" align="bottom-right"/>
-</segment>
-</net>
-<net name="IO27" class="0">
-<segment>
-<pinref part="U$2" gate="G$1" pin="IO27"/>
-<wire x1="-27.94" y1="-10.16" x2="-35.56" y2="-10.16" width="0.1524" layer="91"/>
-<label x="-38.1" y="-10.16" size="1.778" layer="95" align="bottom-right"/>
-</segment>
-</net>
-<net name="IO4" class="0">
-<segment>
-<pinref part="U$2" gate="G$1" pin="IO4"/>
-<wire x1="25.4" y1="-12.7" x2="35.56" y2="-12.7" width="0.1524" layer="91"/>
-<label x="38.1" y="-12.7" size="1.778" layer="95"/>
-</segment>
-</net>
-<net name="IO19" class="0">
-<segment>
-<pinref part="U$2" gate="G$1" pin="IO19"/>
-<wire x1="25.4" y1="0" x2="35.56" y2="0" width="0.1524" layer="91"/>
-<label x="38.1" y="0" size="1.778" layer="95"/>
 </segment>
 </net>
@@
 </segment>
 </net>
-<net name="IO33" class="0">
+<net name="GPIO33" class="0">
+<segment>
+<pinref part="JP7" gate="A" pin="5"/>
+<wire x1="66.04" y1="96.52" x2="55.88" y2="96.52" width="0.1524" layer="91"/>
+<label x="53.34" y="96.52" size="1.778" layer="95" align="bottom-right"/>
+</segment>
+</net>
+<net name="GPIO25" class="0">
+<segment>
+<pinref part="JP7" gate="A" pin="7"/>
+<wire x1="66.04" y1="93.98" x2="55.88" y2="93.98" width="0.1524" layer="91"/>
+<label x="53.34" y="93.98" size="1.778" layer="95" align="bottom-right"/>
+</segment>
+</net>
+<net name="GPIO4" class="0">
+<segment>
+<pinref part="JP7" gate="A" pin="6"/>
+<wire x1="73.66" y1="96.52" x2="83.82" y2="96.52" width="0.1524" layer="91"/>
+<label x="86.36" y="96.52" size="1.778" layer="95"/>
+</segment>
+</net>
+<net name="GPIO16" class="0">
+<segment>
+<pinref part="JP7" gate="A" pin="4"/>
+<wire x1="73.66" y1="99.06" x2="83.82" y2="99.06" width="0.1524" layer="91"/>
+<label x="86.36" y="99.06" size="1.778" layer="95"/>
+</segment>
+</net>
+<net name="GPIO17" class="0">
+<segment>
+<pinref part="JP7" gate="A" pin="2"/>
+<wire x1="73.66" y1="101.6" x2="83.82" y2="101.6" width="0.1524" layer="91"/>
+<label x="86.36" y="101.6" size="1.778" layer="95"/>
+</segment>
+</net>
+<net name="GPIO32" class="0">
 <segment>
 <pinref part="JP7" gate="A" pin="3"/>
@@
 </segment>
 </net>
-<net name="IO27" class="0">
+<net name="GPIO26" class="0">
 <segment>
 <pinref part="JP7" gate="A" pin="9"/>
@@
 </segment>
 </net>
-<net name="IO25" class="0">
-<segment>
-<pinref part="JP7" gate="A" pin="5"/>
-<wire x1="66.04" y1="96.52" x2="55.88" y2="96.52" width="0.1524" layer="91"/>
-<label x="53.34" y="96.52" size="1.778" layer="95" align="bottom-right"/>
-</segment>
-</net>
-<net name="IO26" class="0">
-<segment>
-<pinref part="JP7" gate="A" pin="7"/>
-<wire x1="66.04" y1="93.98" x2="55.88" y2="93.98" width="0.1524" layer="91"/>
-<label x="53.34" y="93.98" size="1.778" layer="95" align="bottom-right"/>
-</segment>
-</net>
-<net name="IO17" class="0">
-<segment>
-<pinref part="JP7" gate="A" pin="6"/>
-<wire x1="73.66" y1="96.52" x2="83.82" y2="96.52" width="0.1524" layer="91"/>
-<label x="86.36" y="96.52" size="1.778" layer="95"/>
-</segment>
-</net>
-<net name="IO4" class="0">
+<net name="GPIO27" class="0">
 <segment>
 <pinref part="JP7" gate="A" pin="8"/>
@@
 </segment>
 </net>
-<net name="IO16" class="0">
-<segment>
-<pinref part="JP7" gate="A" pin="4"/>
-<wire x1="73.66" y1="99.06" x2="83.82" y2="99.06" width="0.1524" layer="91"/>
-<label x="86.36" y="99.06" size="1.778" layer="95"/>
-</segment>
-</net>
-<net name="IO19" class="0">
-<segment>
-<pinref part="JP7" gate="A" pin="2"/>
-<wire x1="73.66" y1="101.6" x2="83.82" y2="101.6" width="0.1524" layer="91"/>
-<label x="86.36" y="101.6" size="1.778" layer="95"/>
-</segment>
-</net>

Commit message: Tweaked and confirmed some connections
Parts:
- removed JP5: LED Type, jumper:JP2E
- removed JP6: JTAG Enable, jumper:JP2E
- added JP3: JTAG, pinhead:PINHD-2X3
- JP1: value JTAG -> 3-pin LED strip; device pinhead:PINHD-1X6 -> pinhead:PINHD-1X3/90
- JP4: value LED Strip -> 4-pin LED Strip
Connections:
- removed net N$7: JP4.3, JP5.2
- removed net TRST_N: JP1.1, JP6.1
- net EN: now also JP3.1; no longer JP6.2, JP6.3
- net GND: now also JP1.1, JP3.6; no longer JP1.6, JP5.1
- net N$8: now also JP1.2, JP4.3; no longer JP4.2
- net N$9: now also JP4.2; no longer JP5.3
- net TCK: now also JP3.4; no longer JP1.4
- net TDI: now also JP3.3; no longer JP1.3
- net TDO: now also JP3.2; no longer JP1.2
- net TMS: now also JP3.5; no longer JP1.5
- net VCC: now also JP1.3
Other:
- moved on the sheet: JP4
