File: hub.brd (EAGLE design)
At the start: 160 x 100 mm, 27 parts, among them U1 10118194-MICRO-USB, U2 LM3671MF-3.3/NOPBMF05A-M, U3 SN74LVC1T45DBVRDBV6-M, U4 SN74LVC1T45DBVRDBV6-M

Commit message: Finished layout!
Connections:
- net TCK: now also JP3.3; no longer JP3.4
- net TDI: now also JP3.4; no longer JP3.3
Routing:
- net CENTER: track 3.15 -> 76.4 mm, vias 0 -> 3
- net EN: track 14.3 -> 61.3 mm, vias 0 -> 3
- net DOWN: track 13.5 -> 55.8 mm, vias 0 -> 1
- net UP: track 7.54 -> 49.6 mm, vias 0 -> 1
- net LED_DATA: track 0.00 -> 34.8 mm, vias 0 -> 2
- net TXD: track 0.00 -> 33.8 mm, vias 0 -> 1
- net TDO: track 0.00 -> 33.3 mm
- net RXD: track 0.00 -> 32.4 mm, vias 0 -> 1
- net GPIO32: track 0.00 -> 28.9 mm, vias 0 -> 1
- net TCK: track 0.00 -> 27.7 mm
- net SDA: track 0.00 -> 27.5 mm, vias 0 -> 1
- net LED_CLOCK: track 0.00 -> 27.0 mm, vias 0 -> 2
- net GPIO33: track 0.00 -> 26.6 mm, vias 0 -> 1
- net GPIO25: track 0.00 -> 24.2 mm, vias 0 -> 1
- net SCL: track 0.00 -> 23.2 mm, vias 0 -> 1
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
Commit message: Final tweaks and BOM creation
Parts:
- renumbered U$1 to U5, U$4 to U6
Other:
- board size 160 x 100 mm -> 46.3 x 36.8 mm
- board text added: "RVL Controller v1.0 Copyright Bryan Hughes October 2019"
