File: ESP.kicad_sch (KiCad schematic)
At the start: 5 parts

Commit message: Bug fix
Parts:
- added C1: 1uF, controller:C0805, symbol controller-eagle-import:C-USC0805
Connections:
- net GND: now also C1.2
- net at R3.1, S3.3, S3.4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: now also C1.1
Other:
- moved on the sheet: R3, S3
