File: controller.kicad_pcb (KiCad board)
At the start: 4 copper layers, 42.8 x 35.9 mm, 28 parts, among them J1 CONN_04SCREW, U1 10118194-MICRO-USB, U2 LM3671MF-3.3/NOPBMF05A-M, U3 SN74LVC1T45DBVRDBV6-M, U4 SN74LVC1T45DBVRDBV6-M

Commit message: Bug fix
Parts:
- added C3: 1uF, controller:C0805, B.Cu at (159.5, 89.6)
Routing:
- net Net-(U$2-EN): track 33.9 -> 36.1 mm
- net GND: track 34.7 -> 36.1 mm, vias 37 -> 38
Other:
- board text added: "RVL Controller v1.7 Copyright Bryan Hughes June 2024"
- board text removed: "RVL Controller v1.6 Copyright Bryan Hughes June 2024"
Changed lines of the file:
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@@
       (net 2 "+3.3V") (pinfunction "VCCB") (pintype "power_in") (solder_mask_margin 0.0635) (thermal_bridge_angle 0))
+  )
+  (footprint "controller:C0805" (layer "B.Cu")
+    (at 159.512 89.601 90)
+    (descr "<b>CAPACITOR</b><p>")
+    (property "Sheetfile" "ESP.kicad_sch")
+    (property "Sheetname" "ESP")
+    (fp_text reference "C3" (at -2.728 -0.508) (layer "B.SilkS")
+        (effects (font (size 0.65532 0.65532) (thickness 0.16383) bold) (justify right bottom mirror))
+    )
+    (fp_text value "1uF" (at -1.27 -2.54 90) (layer "B.Fab")
+        (effects (font (size 1.1684 1.1684) (thickness 0.1016)) (justify right bottom mirror))
+    )
+    (fp_poly
+      (pts
+        (xy -0.1001 -0.4001)
+        (xy 0.1001 -0.4001)
+        (xy 0.1001 0.4001)
+        (xy -0.1001 0.4001)
+      )
+      (stroke (width 0) (type default)) (fill solid) (layer "B.Adhes"))
+    (fp_line (start -1.973 -0.983) (end -1.973 0.983)
+      (stroke (width 0.0508) (type solid)) (layer "B.CrtYd"))
+    (fp_line (start -1.973 0.983) (end 1.973 0.983)
+      (stroke (width 0.0508) (type solid)) (layer "B.CrtYd"))
+    (fp_line (start 1.973 -0.983) (end -1.973 -0.983)
+      (stroke (width 0.0508) (type solid)) (layer "B.CrtYd"))
+    (fp_line (start 1.973 0.983) (end 1.973 -0.983)
+      (stroke (width 0.0508) (type solid)) (layer "B.CrtYd"))
+    (fp_line (start -0.381 0.66) (end 0.381 0.66)
+      (stroke (width 0.1016) (type solid)) (layer "B.Fab"))
+    (fp_line (start -0.356 -0.66) (end 0.381 -0.66)
+      (stroke (width 0.1016) (type solid)) (layer "B.Fab"))
+    (fp_poly
+      (pts
+        (xy -1.0922 -0.7239)
+        (xy -0.3421 -0.7239)
+        (xy -0.3421 0.7262)
+        (xy -1.0922 0.7262)
+      )
+      (stroke (width 0) (type default)) (fill solid) (layer "B.Fab"))
+    (fp_poly
+      (pts
+        (xy 0.3556 -0.7239)
+        (xy 1.1057 -0.7239)
+        (xy 1.1057 0.7262)
+        (xy 0.3556 0.7262)
+      )
+      (stroke (width 0) (type default)) (fill solid) (layer "B.Fab"))
+    (pad "1" smd rect (at -0.95 0 90) (size 1.3 1.5) (layers "B.Cu" "B.Paste" "B.Mask")
+      (net 32 "Net-(U$2-EN)") (pinfunction "1") (pintype "passive") (solder_mask_margin 0.0635) (thermal_bridge_angle 0))
+    (pad "2" smd rect (at 0.95 0 90) (size 1.3 1.5) (layers "B.Cu" "B.Paste" "B.Mask")
+      (net 1 "GND") (pinfunction "2") (pintype "passive") (solder_mask_margin 0.0635) (thermal_bridge_angle 0))
   )
   (footprint "controller:R0805" (layer "B.Cu")
@@
     (property "Sheetfile" "ESP.kicad_sch")
     (property "Sheetname" "ESP")
-    (fp_text reference "R3" (at 0.6986 2.01565 90) (layer "B.SilkS")
+    (fp_text reference "R3" (at -2.7304 0.74565 180) (layer "B.SilkS")
         (effects (font (size 0.65532 0.65532) (thickness 0.23368)) (justify left bottom mirror))
     )
@@
     (effects (font (size 0.7112 0.7112) (thickness 0.1778)) (justify left top mirror))
   )
-  (gr_text "RVL Controller v1.6\nCopyright Bryan Hughes\nJune 2024" (at 127.39735 101.6636 270) (layer "B.SilkS")
+  (gr_text "RVL Controller v1.7\nCopyright Bryan Hughes\nJune 2024" (at 127.39735 101.6636 270) (layer "B.SilkS")
     (effects (font (size 0.7112 0.7112) (thickness 0.1778)) (justify left bottom mirror))
   )
@@
   (via (at 144.85985 95.6311) (size 0.5532) (drill 0.35) (layers "F.Cu" "B.Cu") (net 1))
   (via (at 134.38235 103.8861) (size 0.5532) (drill 0.35) (layers "F.Cu" "B.Cu") (net 1))
+  (via (at 160.909 88.646) (size 0.6) (drill 0.3) (layers "F.Cu" "B.Cu") (net 1))
   (via (at 168.35485 104.2036) (size 0.5532) (drill 0.35) (layers "F.Cu" "B.Cu") (net 1))
   (segment (start 150.57485 105.5211) (end 150.57485 107.0611) (width 0.6096) (layer "B.Cu") (net 1))
@@
   (segment (start 152.58145 108.9661) (end 154.16895 108.9661) (width 0.3048) (layer "B.Cu") (net 1))
   (segment (start 145.85985 95.6311) (end 145.81235 95.6786) (width 0.6096) (layer "B.Cu") (net 1))
+  (segment (start 160.904 88.651) (end 160.909 88.646) (width 0.2) (layer "B.Cu") (net 1))
   (segment (start 145.81235 95.6786) (end 145.81235 96.5836) (width 0.6096) (layer "B.Cu") (net 1))
+  (segment (start 159.512 88.651) (end 160.904 88.651) (width 0.2) (layer "B.Cu") (net 1))
   (segment (start 156.50575 108.9661) (end 158.09325 108.9661) (width 0.3048) (layer "B.Cu") (net 1))
   (segment (start 154.16895 114.0461) (end 156.50575 114.0461) (width 0.3048) (layer "B.Cu") (net 1))
@@
   (segment (start 157.56235 90.8686) (end 157.24235 90.5486) (width 0.3048) (layer "B.Cu") (net 32))
   (segment (start 153.35985 90.5511) (end 141.36735 90.5511) (width 0.3048) (layer "B.Cu") (net 32))
+  (segment (start 159.5096 90.5486) (end 159.512 90.551) (width 0.3048) (layer "B.Cu") (net 32))
+  (segment (start 157.24235 90.5486) (end 159.5096 90.5486) (width 0.3048) (layer "B.Cu") (net 32))
   (segment (start 141.36735 90.5511) (end 140.09735 89.2811) (width 0.3048) (layer "B.Cu") (net 32))
   (segment (start 132.62235 99.9036) (end 132.6361 99.91735) (width 0.3048) (layer "F.Cu") (net 33))
