File: receiver/Extension_Headers.kicad_sch (KiCad schematic)
At the start: 7 parts, among them U5 FT231XQ-R, U6 MBT3904DW1T1G

Commit message: First draft of new receiver
Parts:
- U5: footprint FT231XQ-R:QFN50P400X400X80-21N -> receiver:QFN50P400X400X80-21N
- U6: footprint MBT3904DW1T1G:SOT236 -> receiver:SOT236
Changed lines of the file:
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@@
 			)
 		)
-		(property "Footprint" "MBT3904DW1T1G:SOT236"
+		(property "Footprint" "receiver:SOT236"
 			(at 226.06 121.92 0)
 			(effects
@@
 			)
 		)
-		(property "Footprint" "FT231XQ-R:QFN50P400X400X80-21N"
+		(property "Footprint" "receiver:QFN50P400X400X80-21N"
 			(at 166.37 121.92 0)
 			(effects

Commit message: Finished first draft of new receiver
Parts:
- U6: footprint receiver:SOT236 -> MBT3904DW1T1G:SOT236
Changed lines of the file:
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@@
 			)
 		)
-		(property "Footprint" "receiver:SOT236"
+		(property "Footprint" "MBT3904DW1T1G:SOT236"
 			(at 226.06 121.92 0)
 			(effects
