File: receiver/Extension_Headers.kicad_sch (KiCad schematic)
At the start: 7 parts, among them U5 FT231XQ-R, U6 MBT3904DW1T1G

Commit message: Started redesigning receiver
Parts:
- U6: footprint MBT3904DW1T1G:SOT236 -> receiver:SOT236
Changed lines of the file:
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@@
 			)
 		)
-		(property "Footprint" "MBT3904DW1T1G:SOT236"
+		(property "Footprint" "receiver:SOT236"
 			(at 226.06 121.92 0)
 			(effects
